File: 2024-03-18_driver_nema17/kicad7/nema17_driver/nema17_driver.kicad_pcb (KiCad board)
At the start: 2 copper layers, 42.4 x 42.4 mm, 47 parts, among them U1 AS5600, U2 SP3485CN, U3 STM32C031C6T6, X1 IN, X2 OUT, X3 MOTOR, X4 JTAG, X5 DEBUG

Commit message: Gerber
Parts:
- added G***: LOGO, MyLib:logo-progetti, B.Cu at (161.4, 82.6)
- X1, X2: footprint Connector_PinSocket_2.54mm:PinSocket_1x04_P2.54mm_Vertical -> Connector_PinHeader_2.54mm:PinHeader_1x04_P2.54mm_Vertical
- moved R4 5.15 mm to (138.4, 71.0)
- moved R2 5.01 mm to (143.5, 71.1)
- moved U2 0.85 mm to (129.3, 87.6)
- moved C4 0.64 mm to (146.6, 89.4)
- moved R6 0.39 mm to (148.4, 65.4)
- moved R5 0.36 mm to (153.6, 65.4)
- moved JP1 0.32 mm to (136.2, 87.9)
Connections:
- C5 pad 1: +3V3 -> +3.3V
- JP10 pad 1: +3V3 -> +3.3V
- JP3 pad 1: +3V3 -> +3.3V
- JP4 pad 1: +3V3 -> +3.3V
- JP5 pad 1: +3V3 -> +3.3V
- JP6 pad 1: +3V3 -> +3.3V
- JP7 pad 1: +3V3 -> +3.3V
- JP8 pad 1: +3V3 -> +3.3V
- JP9 pad 1: +3V3 -> +3.3V
- R10 pad 2: Net-(U3-PA7) -> Net-(U3-PB0)
- R11 pad 2: Net-(U3-PB0) -> Net-(U3-PA7)
- R12 pad 2: Net-(U3-PB1) -> Net-(U3-PA6)
- R13 pad 2: Net-(U3-PB2) -> Net-(U3-PA5)
- R14 pad 2: Net-(U3-PB10) -> Net-(U3-PA4)
- R2 pad 1: +3V3 -> +3.3V
- R3 pad 1: +3V3 -> +3.3V
- R4 pad 1: +3V3 -> +3.3V
- R7 pad 2: Net-(U3-PA4) -> Net-(U3-PB10)
- R8 pad 2: Net-(U3-PA5) -> Net-(U3-PB2)
- R9 pad 2: Net-(U3-PA6) -> Net-(U3-PB1)
- U1 pad 1: +3V3 -> +3.3V
- U1 pad 2: +3V3 -> +3.3V
- U1 pad 8: +3V3 -> +3.3V
- X1 pad 3: Net-(JP1-B) -> Net-(U2-B)
- X1 pad 4: Net-(U2-B) -> Net-(JP1-B)
- X2 pad 3: Net-(JP1-B) -> Net-(U2-B)
- X2 pad 4: Net-(U2-B) -> Net-(JP1-B)
Routing:
- net +3.3V: track 0.00 -> 81.9 mm, vias 0 -> 4
- net Net-(JP1-B): track 0.00 -> 53.1 mm, vias 0 -> 1
- net +12V: track 0.00 -> 43.6 mm
- net U2-TX-DCE: track 0.00 -> 41.9 mm, vias 0 -> 2
- net Net-(U3-PB10): track 0.00 -> 38.6 mm
- net Net-(U2-B): track 0.00 -> 37.7 mm
- net Net-(U3-PB2): track 0.00 -> 34.7 mm
- net SWCLK: track 0.00 -> 33.3 mm, vias 0 -> 1
- net Net-(U3-PB1): track 0.00 -> 31.3 mm
- net SWDIO: track 0.00 -> 31.3 mm, vias 0 -> 1
- net Net-(U3-PB0): track 0.00 -> 27.8 mm
- net Net-(U3-PA7): track 0.00 -> 24.4 mm
- net Net-(U3-PA6): track 0.00 -> 21.0 mm
- net Net-(POW2-Pin_3): track 0.00 -> 18.5 mm
- net Net-(U3-PA5): track 0.00 -> 17.6 mm
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- added copper zone on F.Cu, net +3.3V
- added copper zone on B.Cu, net GND
- added copper zone on F.Cu, net GND
Other:
- board text added: "+12V G B A"
- board text added: "GND TX RX"
- board text added: "NEMA17 DRIVER"
- board text added: "bottom"
