File: 2024-09-16_mangiatoia_automatica/2_pcb-mangiatoia/kicad7/mangiatoia.kicad_pcb (KiCad board)
At the start: 2 copper layers, 140 x 80 mm, 43 parts, among them J1 POWER, J2 FEED, J3 SERVO, J4 GPIO, J5 L-CELL, J6 L-CELL, J7 L-CELL, K1 FINDER-36.11, Q1 BC817, U1 ESP32-DevKitC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

Commit message: v1.1
Connections:
- J5 pad 1: +5V -> +3.3V
Routing:
- net +3.3V: track 102.9 -> 123.8 mm, vias 2 -> 3
- net SCK: track 120.0 -> 125.3 mm
- net MOSI: track 112.8 -> 117.8 mm
- net +5V: track 214.8 -> 217.0 mm
- net SD-CS: track 76.1 -> 77.6 mm
- net TFT-LED: track 31.8 -> 33.0 mm
- net TFT-CS: track 38.8 -> 37.6 mm
- net TOUCH-CS: track 31.6 -> 32.7 mm
- net TFT-DC: track 22.6 -> 23.5 mm
Other:
- board text added: "MAEDC v1.1"
- board text removed: "MAEDC v1.0"

Commit message: debug 485
Other:
- board text added: "+12V GND"
- board text added: "A B GND +12V"
- board text added: "GND +5 PWM"
- board text added: "GND IN"
Changed lines of the file:
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@@
     (effects (font (size 1 1) (thickness 0.15)) (justify left bottom))
+  )
+  (gr_text "+12V\n\n\n\n\n\n\nGND" (at 80.157572 109.122155) (layer "F.SilkS")
+    (effects (font (size 0.8 0.75) (thickness 0.1)) (justify left bottom))
   )
   (gr_text "GPIO" (at 72.062 60.071 270) (layer "F.SilkS")
     (effects (font (size 1 1) (thickness 0.15)) (justify left bottom))
+  )
+  (gr_text "GND\n\n+5\n\nPWM" (at 78.387239 78.201647) (layer "F.SilkS")
+    (effects (font (size 0.8 0.75) (thickness 0.1)) (justify left bottom))
+  )
+  (gr_text "GND\n\nIN" (at 78.519706 64.135) (layer "F.SilkS")
+    (effects (font (size 0.8 0.75) (thickness 0.1)) (justify left bottom))
   )
   (gr_text "MAEDC v1.1" (at 179.25 57.531) (layer "F.SilkS")
@@
     (effects (font (size 1 1) (thickness 0.15)) (justify left bottom))
   )
+  (gr_text "A\n\nB\n\nGND\n\n+12V" (at 78.519706 93.372017) (layer "F.SilkS")
+    (effects (font (size 0.8 0.75) (thickness 0.1)) (justify left bottom))
+  )
   (dimension (type aligned) (layer "F.Fab")

Commit message: memory heap
Parts:
- added BZ1: Buzzer, Buzzer_Beeper:Buzzer_12x9.5RM7.6, F.Cu at (99.7, 118.4)
- moved R5 0.88 mm to (103.9, 120.0)
Routing:
- net /LED: track 4.80 -> 7.50 mm
- net Net-(U1-32K_XP/GPIO32/ADC1_CH4): track 82.1 -> 81.2 mm
Changed lines of the file:
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@@
     )
   )
+  (footprint "Buzzer_Beeper:Buzzer_12x9.5RM7.6" (layer "F.Cu")
+    (at 99.748 118.364 180)
+    (descr "Generic Buzzer, D12mm height 9.5mm with RM7.6mm")
+    (tags "buzzer")
+    (property "Sheetfile" "mangiatoia.kicad_sch")
+    (property "Sheetname" "")
+    (property "ki_description" "Buzzer, polarized")
+    (property "ki_keywords" "quartz resonator ceramic")
+    (attr through_hole)
+    (fp_text reference "BZ1" (at 9.779 5.08) (layer "F.SilkS")
+        (effects (font (size 1 1) (thickness 0.15)))
+    )
+    (fp_text value "Buzzer" (at 3.8 7.4) (layer "F.Fab")
+        (effects (font (size 1 1) (thickness 0.15)))
+    )
+    (fp_text user "+" (at -0.01 -2.54) (layer "F.SilkS")
+        (effects (font (size 1 1) (thickness 0.15)))
+    )
+    (fp_text user "+" (at -0.01 -2.54) (layer "F.Fab")
+        (effects (font (size 1 1) (thickness 0.15)))
+    )
+    (fp_text user "${REFERENCE}" (at 3.8 -4) (layer "F.Fab")
+        (effects (font (size 1 1) (thickness 0.15)))
+    )
+    (fp_circle (center 3.8 0) (end 9.9 0)
+      (stroke (width 0.12) (type solid)) (fill none) (layer "F.SilkS"))
+    (fp_circle (center 3.8 0) (end 10.05 0)
+      (stroke (width 0.05) (type solid)) (fill none) (layer "F.CrtYd"))
+    (fp_circle (center 3.8 0) (end 4.8 0)
+      (stroke (width 0.1) (type solid)) (fill none) (layer "F.Fab"))
+    (fp_circle (center 3.8 0) (end 9.8 0)
+      (stroke (width 0.1) (type solid)) (fill none) (layer "F.Fab"))
+    (pad "1" thru_hole rect (at 0 0 180) (size 2 2) (drill 1) (layers "*.Cu" "*.Mask")
+      (net 5 "/LED") (pinfunction "-") (pintype "passive"))
+    (pad "2" thru_hole circle (at 7.6 0 180) (size 2 2) (drill 1) (layers "*.Cu" "*.Mask")
+      (net 2 "GND") (pinfunction "+") (pintype "passive"))
+    (model "${KICAD6_3DMODEL_DIR}/Buzzer_Beeper.3dshapes/Buzzer_12x9.5RM7.6.wrl"
+      (offset (xyz 0 0 0))
+      (scale (xyz 1 1 1))
+      (rotate (xyz 0 0 0))
+    )
+  )
   (footprint "Capacitor_SMD:C_0603_1608Metric" (layer "F.Cu")
     (at 109.41 111.855)
@@
   )
   (footprint "Resistor_SMD:R_0805_2012Metric" (layer "F.Cu")
-    (at 103.06 120.095)
+    (at 103.939 120.015)
     (descr "Resistor SMD 0805 (2012 Metric), square (rectangular) end terminal, IPC_7351 nominal, (Body size source: IPC-SM-782 page 72, https://www.pcb-3d.com/wordpress/wp-content/uploads/ipc-sm-782a_amendment_1_and_2.pdf), generated with kicad-footprint-generator")
     (tags "resistor")
@@
   (segment (start 135.255 96.34) (end 135.255 97.155) (width 0.6096) (layer "B.Cu") (net 4))
   (segment (start 134.546 77.851) (end 133.53 78.867) (width 0.6096) (layer "B.Cu") (net 4))
-  (segment (start 97.345 120.095) (end 102.1475 120.095) (width 0.6096) (layer "F.Cu") (net 5))
+  (segment (start 102.9465 120.095) (end 103.0265 120.015) (width 0.6096) (layer "F.Cu") (net 5))
+  (segment (start 99.748 118.364) (end 99.621 118.491) (width 0.6096) (layer "F.Cu") (net 5))
+  (segment (start 97.345 120.095) (end 99.621 120.095) (width 0.6096) (layer "F.Cu") (net 5))
+  (segment (start 99.621 118.491) (end 99.621 120.095) (width 0.6096) (layer "F.Cu") (net 5))
+  (segment (start 99.621 120.095) (end 102.9465 120.095) (width 0.6096) (layer "F.Cu") (net 5))
   (segment (start 111.315 68.3425) (end 111.315 69.723) (width 0.6096) (layer "F.Cu") (net 6))
   (segment (start 84.7165 62.611) (end 84.645 62.6825) (width 0.6096) (layer "F.Cu") (net 6))
@@
   (segment (start 117.274 95.631) (end 120.068 98.425) (width 0.6096) (layer "B.Cu") (net 15))
   (segment (start 117.02 97.917) (end 117.02 96.393) (width 0.4064) (layer "F.Cu") (net 16))
-  (segment (start 103.9725 120.095) (end 106.272 120.095) (width 0.4064) (layer "F.Cu") (net 16))
+  (segment (start 104.8515 120.015) (end 106.352 120.015) (width 0.4064) (layer "F.Cu") (net 16))
   (segment (start 117.02 96.393) (end 117.782 95.631) (width 0.4064) (layer "F.Cu") (net 16))
   (segment (start 132.419 92.17) (end 163.385 92.17) (width 0.4064) (layer "F.Cu") (net 16))
-  (segment (start 106.272 120.095) (end 106.352 120.015) (width 0.4064) (layer "F.Cu") (net 16))
   (segment (start 117.782 95.631) (end 128.958 95.631) (width 0.4064) (layer "F.Cu") (net 16))
   (segment (start 128.958 95.631) (end 132.419 92.17) (width 0.4064) (layer "F.Cu") (net 16))
