File: 2024-09-16_mangiatoia_automatica/2_pcb-mangiatoia/kicad7/mangiatoia.kicad_sch (KiCad schematic)
At the start: 40 parts, among them J1 POWER, J2 FEED, J3 SERVO, J4 GPIO, J5 L-CELL, J6 L-CELL, J7 L-CELL, K1 FINDER-36.11, Q1 BC817, U1 ESP32-DevKitC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

Commit message: TEST PCB
Parts:
- U1: Buy (none) -> https://amzn.to/4eelbHS
Other:
- note added: "ERRORE QUI VA 3,3V!"
Changed lines of the file:
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@@
     (effects (font (size 1.5 1.5)) (justify right bottom))
+  )
+  (text "ERRORE\nQUI VA\n3,3V!" (at 113.03 120.65 0)
+    (effects (font (size 1.27 1.27) (thickness 0.254) bold (color 194 0 0 1)) (justify left bottom))
   )
   (text "PULL-UP e \nPULL-DOWN\nSUL MASTER" (at 111.76 169.545 0)
@@
     )
     (property "Datasheet" "https://docs.espressif.com/projects/esp-idf/zh_CN/latest/esp32/hw-reference/esp32/get-started-devkitc.html" (at 102.235 111.76 0)
+      (effects (font (size 1.27 1.27)) hide)
+    )
+    (property "Buy" "https://amzn.to/4eelbHS" (at 102.235 66.04 0)
+      (effects (font (size 1.27 1.27)) hide)
+    )
+    (property "Campo5" "" (at 102.235 66.04 0)
       (effects (font (size 1.27 1.27)) hide)
     )
@@
       (effects (font (size 1.27 1.27) italic) (justify left) hide)
     )
-    (property "Datasheet" "http://www.st.com/content/ccc/resource/technical/document/datasheet/41/4f/b3/b0/12/d4/47/88/CD00000444.pdf/files/CD00000444.pdf/jcr:content/translations/en.CD00000444.pdf" (at 68.58 138.43 0)
+    (property "Datasheet" "https://www.mouser.it/ProductDetail/MEAN-WELL/N7805-1C?qs=7D1LtPJG0i2aXH7i3d%252BGOw%3D%3D" (at 68.58 138.43 0)
+      (effects (font (size 1.27 1.27)) hide)
+    )
+    (property "Campo4" "" (at 68.58 137.16 0)
       (effects (font (size 1.27 1.27)) hide)
     )
@@
       (effects (font (size 1.27 1.27)) hide)
     )
-    (property "Datasheet" "http://power.murata.com/datasheet?/data/power/ncl/kdc_cre1.pdf" (at 68.58 133.35 0)
-      (effects (font (size 1.27 1.27)) hide)
-    )
+    (property "Datasheet" "https://amzn.to/3AqUi5z" (at 68.58 133.35 0)
+      (effects (font (size 1.27 1.27)) hide)
+    )

Commit message: v1.1
Connections:
- net +3.3V: now also J5.1 (Pin_1)
- net +5V: no longer J5.1 (Pin_1)
Other:
- note added: "+3,3 SCK DT GND"
- note added: "HX711"
- note removed: "+5 SCK DT GND"
- note removed: "ERRORE QUI VA 3,3V!"
Changed lines of the file:
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@@
   (title_block
     (title "Mangiatoia per animali domestici ")
-    (date "2024-09-21")
-    (rev "1.0")
+    (date "2024-11-06")
+    (rev "1.1")
     (company "PROGETTI di Frisoni Emanuele")
   )
@@
     (stroke (width 0) (type default))
   )
-  (wire (pts (xy 123.825 128.27) (xy 123.825 132.08))
+  (wire (pts (xy 124.46 128.27) (xy 124.46 132.08))
     (stroke (width 0) (type default))
   )
@@
     (stroke (width 0) (type default))
   )
-  (wire (pts (xy 128.905 128.27) (xy 123.825 128.27))
+  (wire (pts (xy 128.905 128.27) (xy 124.46 128.27))
     (stroke (width 0) (type default))
   )
@@
     (stroke (width 0) (type default))
   )
-  (wire (pts (xy 128.905 120.65) (xy 123.825 120.65))
+  (wire (pts (xy 128.905 120.65) (xy 124.46 120.65))
     (stroke (width 0) (type default))
   )
@@
     (stroke (width 0) (type default))
   )
-  (wire (pts (xy 123.825 120.65) (xy 123.825 118.11))
+  (wire (pts (xy 124.46 120.65) (xy 124.46 118.11))
     (stroke (width 0) (type default))
   )
@@
     (effects (font (size 1.27 1.27)) (justify left bottom))
   )
-  (text "+5\nSCK\nDT\nGND" (at 140.335 128.27 0)
+  (text "+3,3\nSCK\nDT\nGND" (at 140.335 128.27 0)
     (effects (font (size 1.5 1.5)) (justify right bottom))
   )
-  (text "ERRORE\nQUI VA\n3,3V!" (at 113.03 120.65 0)
-    (effects (font (size 1.27 1.27) (thickness 0.254) bold (color 194 0 0 1)) (justify left bottom))
-  )
   (text "PULL-UP e \nPULL-DOWN\nSUL MASTER" (at 111.76 169.545 0)
     (effects (font (size 1.27 1.27)) (justify right bottom))
@@
     (effects (font (size 1.5 1.5)) (justify left bottom))
   )
+  (text "HX711" (at 144.78 116.84 0)
+    (effects (font (size 2 2)) (justify left bottom))
+  )
   (text "input\nonly" (at 43.18 66.04 0)
     (effects (font (size 1.27 1.27)) (justify right bottom))
@@
     )
   )
-  (symbol (lib_id "power:+5V") (at 123.825 118.11 0) (mirror y) (unit 1)
-    (in_bom yes) (on_board yes) (dnp no) (fields_autoplaced)
-    (property "Reference" "#PWR026" (at 123.825 121.92 0)
-      (effects (font (size 1.27 1.27)) hide)
-    )
-    (property "Value" "+5V" (at 123.825 114.3 0)
-      (effects (font (size 1.27 1.27)))
-    )
-    (property "Footprint" "" (at 123.825 118.11 0)
-      (effects (font (size 1.27 1.27)) hide)
-    )
-    (property "Datasheet" "" (at 123.825 118.11 0)
-      (effects (font (size 1.27 1.27)) hide)
-    )
-    (pin "1")
-    (instances
-      (project "mangiatoia"
-        (path "/4dc09dc3-e9dc-41d7-affd-028107848572"
-          (reference "#PWR026") (unit 1)
-        )
-      )
-    )
-  )
   (symbol (lib_id "Connector:Screw_Terminal_01x02") (at 26.035 123.19 0) (mirror y) (unit 1)
     (in_bom yes) (on_board yes) (dnp no) (fields_autoplaced)
@@
     )
   )
+  (symbol (lib_id "power:+3.3V") (at 124.46 118.11 0) (unit 1)
+    (in_bom yes) (on_board yes) (dnp no) (fields_autoplaced)
+    (property "Reference" "#PWR026" (at 124.46 121.92 0)
+      (effects (font (size 1.27 1.27)) hide)
+    )
+    (property "Value" "+3.3V" (at 124.46 114.3 0)
+      (effects (font (size 1.27 1.27)))
+    )
+    (property "Footprint" "" (at 124.46 118.11 0)
+      (effects (font (size 1.27 1.27)) hide)
+    )
+    (property "Datasheet" "" (at 124.46 118.11 0)
+      (effects (font (size 1.27 1.27)) hide)
+    )
+    (pin "1")
+    (instances
+      (project "mangiatoia"
+        (path "/4dc09dc3-e9dc-41d7-affd-028107848572"
+          (reference "#PWR026") (unit 1)
+        )
+      )
+    )
+  )
   (symbol (lib_id "Transistor_BJT:BC817") (at 222.885 140.335 0) (unit 1)
     (in_bom yes) (on_board yes) (dnp no)
@@
     )
   )
-  (symbol (lib_id "power:GND") (at 123.825 132.08 0) (mirror y) (unit 1)
+  (symbol (lib_id "power:GND") (at 124.46 132.08 0) (mirror y) (unit 1)
     (in_bom yes) (on_board yes) (dnp no)
-    (property "Reference" "#PWR027" (at 123.825 138.43 0)
+    (property "Reference" "#PWR027" (at 124.46 138.43 0)
       (effects (font (size 1.27 1.27)) hide)
     )
-    (property "Value" "GND" (at 123.825 136.525 0)
+    (property "Value" "GND" (at 124.46 136.525 0)
       (effects (font (size 1.27 1.27)))
     )
-    (property "Footprint" "" (at 123.825 132.08 0)
+    (property "Footprint" "" (at 124.46 132.08 0)
       (effects (font (size 1.27 1.27)) hide)
     )
-    (property "Datasheet" "" (at 123.825 132.08 0)
+    (property "Datasheet" "" (at 124.46 132.08 0)
       (effects (font (size 1.27 1.27)) hide)
     )

Commit message: memory heap
Parts:
- added BZ1: Buzzer, Buzzer_Beeper:Buzzer_12x9.5RM7.6, symbol Device:Buzzer
Connections:
- net GND: now also BZ1.2 (+)
- net LED: now also BZ1.1 (-)
Other:
- moved on the sheet: C1, DL1
Changed lines of the file:
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@@
   (junction (at 225.425 152.4) (diameter 0) (color 0 0 0 0)
   )
+  (junction (at 30.48 53.975) (diameter 0) (color 0 0 0 0)
+  )
+  (junction (at 34.29 40.64) (diameter 0) (color 0 0 0 0)
+  )
   (junction (at 215.265 140.335) (diameter 0) (color 0 0 0 0)
   )
@@
     (stroke (width 0) (type default))
   )
-  (wire (pts (xy 33.655 55.245) (xy 33.655 50.8))
-    (stroke (width 0) (type default))
-  )
   (wire (pts (xy 247.015 47.625) (xy 247.015 48.895))
     (stroke (width 0) (type default))
@@
     (stroke (width 0) (type default))
   )
+  (wire (pts (xy 36.195 51.435) (xy 34.925 51.435))
+    (stroke (width 0) (type default))
+  )
   (wire (pts (xy 225.425 152.4) (xy 215.265 152.4))
     (stroke (width 0) (type default))
@@
     (stroke (width 0) (type default))
   )
-  (wire (pts (xy 20.955 46.99) (xy 20.955 55.245))
+  (wire (pts (xy 17.78 46.99) (xy 17.78 55.245))
     (stroke (width 0) (type default))
   )
@@
     (stroke (width 0) (type default))
   )
+  (wire (pts (xy 30.48 53.975) (xy 30.48 55.245))
+    (stroke (width 0) (type default))
+  )
   (wire (pts (xy 135.255 71.12) (xy 162.56 71.12))
     (stroke (width 0) (type default))
@@
     (stroke (width 0) (type default))
   )
+  (wire (pts (xy 34.29 46.355) (xy 34.29 40.64))
+    (stroke (width 0) (type default))
+  )
   (wire (pts (xy 69.215 66.04) (xy 62.865 66.04))
     (stroke (width 0) (type default))
@@
     (stroke (width 0) (type default))
   )
+  (wire (pts (xy 34.29 40.64) (xy 46.355 40.64))
+    (stroke (width 0) (type default))
+  )
   (wire (pts (xy 193.04 83.82) (xy 193.04 91.44))
     (stroke (width 0) (type default))
@@
     (stroke (width 0) (type default))
   )
-  (wire (pts (xy 20.955 35.56) (xy 20.955 39.37))
+  (wire (pts (xy 17.78 35.56) (xy 17.78 39.37))
     (stroke (width 0) (type default))
   )
@@
     (stroke (width 0) (type default))
   )
-  (wire (pts (xy 33.655 40.64) (xy 46.355 40.64))
+  (wire (pts (xy 30.48 40.64) (xy 34.29 40.64))
     (stroke (width 0) (type default))
   )
@@
     (stroke (width 0) (type default))
   )
+  (wire (pts (xy 34.925 53.975) (xy 30.48 53.975))
+    (stroke (width 0) (type default))
+  )
   (wire (pts (xy 52.07 176.53) (xy 45.72 176.53))
     (stroke (width 0) (type default))
@@
     (stroke (width 0) (type default))
   )
-  (wire (pts (xy 45.085 35.56) (xy 20.955 35.56))
+  (wire (pts (xy 45.085 35.56) (xy 17.78 35.56))
     (stroke (width 0) (type default))
   )
@@
     (stroke (width 0) (type default))
   )
-  (wire (pts (xy 33.655 40.64) (xy 33.655 43.18))
+  (wire (pts (xy 30.48 40.64) (xy 30.48 43.18))
     (stroke (width 0) (type default))
   )
@@
     (stroke (width 0) (type default))
   )
+  (wire (pts (xy 36.195 46.355) (xy 34.29 46.355))
+    (stroke (width 0) (type default))
+  )
   (wire (pts (xy 135.255 48.26) (xy 146.685 48.26))
     (stroke (width 0) (type default))
@@
     (stroke (width 0) (type default))
   )
+  (wire (pts (xy 34.925 51.435) (xy 34.925 53.975))
+    (stroke (width 0) (type default))
+  )
   (wire (pts (xy 270.51 82.55) (xy 270.51 85.09))
     (stroke (width 0) (type default))
   )
+  (wire (pts (xy 30.48 50.8) (xy 30.48 53.975))
+    (stroke (width 0) (type default))
+  )
   (wire (pts (xy 247.015 48.895) (xy 249.555 48.895))
     (stroke (width 0) (type default))
@@
     )
   )
-  (symbol (lib_id "Device:C_Polarized") (at 20.955 43.18 0) (unit 1)
+  (symbol (lib_id "Device:C_Polarized") (at 17.78 43.18 0) (unit 1)
     (in_bom yes) (on_board yes) (dnp no) (fields_autoplaced)
-    (property "Reference" "C1" (at 24.765 41.656 0)
+    (property "Reference" "C1" (at 21.59 41.656 0)
       (effects (font (size 1.27 1.27)) (justify left))
     )
-    (property "Value" "10uF" (at 24.765 44.196 0)
+    (property "Value" "10uF" (at 21.59 44.196 0)
       (effects (font (size 1.27 1.27)) (justify left))
     )
-    (property "Footprint" "Capacitor_THT:CP_Radial_D6.3mm_P2.50mm" (at 21.9202 46.99 0)
+    (property "Footprint" "Capacitor_THT:CP_Radial_D6.3mm_P2.50mm" (at 18.7452 46.99 0)
       (effects (font (size 1.27 1.27)) hide)
     )
-    (property "Datasheet" "~" (at 20.955 43.18 0)
+    (property "Datasheet" "~" (at 17.78 43.18 0)
       (effects (font (size 1.27 1.27)) hide)
     )
@@
     )
   )
-  (symbol (lib_id "Device:LED") (at 33.655 46.99 90) (unit 1)
+  (symbol (lib_id "Device:LED") (at 30.48 46.99 90) (unit 1)
     (in_bom yes) (on_board yes) (dnp no)
-    (property "Reference" "DL1" (at 32.385 50.8 0)
+    (property "Reference" "DL1" (at 29.21 50.8 0)
       (effects (font (size 1.27 1.27)))
     )
-    (property "Value" "ST" (at 32.385 43.815 0)
+    (property "Value" "ST" (at 29.21 43.815 0)
       (effects (font (size 1.27 1.27)))
     )
-    (property "Footprint" "LED_THT:LED_D5.0mm" (at 33.655 46.99 0)
+    (property "Footprint" "LED_THT:LED_D5.0mm" (at 30.48 46.99 0)
       (effects (font (size 1.27 1.27)) hide)
     )
-    (property "Datasheet" "~" (at 33.655 46.99 0)
+    (property "Datasheet" "~" (at 30.48 46.99 0)
       (effects (font (size 1.27 1.27)) hide)
     )
@@
     )
   )
-  (symbol (lib_id "power:GND") (at 33.655 55.245 0) (unit 1)
+  (symbol (lib_id "power:GND") (at 30.48 55.245 0) (unit 1)
     (in_bom yes) (on_board yes) (dnp no) (fields_autoplaced)
-    (property "Reference" "#PWR02" (at 33.655 61.595 0)
+    (property "Reference" "#PWR02" (at 30.48 61.595 0)
       (effects (font (size 1.27 1.27)) hide)
     )
-    (property "Value" "GND" (at 33.655 60.325 0)
+    (property "Value" "GND" (at 30.48 60.325 0)
       (effects (font (size 1.27 1.27)))
     )
-    (property "Footprint" "" (at 33.655 55.245 0)
+    (property "Footprint" "" (at 30.48 55.245 0)
       (effects (font (size 1.27 1.27)) hide)
     )
-    (property "Datasheet" "" (at 33.655 55.245 0)
+    (property "Datasheet" "" (at 30.48 55.245 0)
       (effects (font (size 1.27 1.27)) hide)
     )
@@
     )
   )
-  (symbol (lib_id "power:GND") (at 20.955 55.245 0) (unit 1)
+  (symbol (lib_id "Device:Buzzer") (at 38.735 48.895 0) (unit 1)
+    (in_bom yes) (on_board yes) (dnp no) (fields_autoplaced)
+    (property "Reference" "BZ1" (at 42.545 48.26 0)
+      (effects (font (size 1.27 1.27)) (justify left))
+    )
+    (property "Value" "Buzzer" (at 42.545 50.8 0)
+      (effects (font (size 1.27 1.27)) (justify left))
+    )
+    (property "Footprint" "Buzzer_Beeper:Buzzer_12x9.5RM7.6" (at 38.1 46.355 90)
+      (effects (font (size 1.27 1.27)) hide)
+    )
+    (property "Datasheet" "~" (at 38.1 46.355 90)
+      (effects (font (size 1.27 1.27)) hide)
+    )
+    (pin "1")
+    (pin "2")
+    (instances
+      (project "mangiatoia"
+        (path "/4dc09dc3-e9dc-41d7-affd-028107848572"
+          (reference "BZ1") (unit 1)
+        )
+      )
+    )
+  )
+  (symbol (lib_id "power:GND") (at 17.78 55.245 0) (unit 1)
     (in_bom yes) (on_board yes) (dnp no) (fields_autoplaced)
-    (property "Reference" "#PWR01" (at 20.955 61.595 0)
+    (property "Reference" "#PWR01" (at 17.78 61.595 0)
       (effects (font (size 1.27 1.27)) hide)
     )
-    (property "Value" "GND" (at 20.955 60.325 0)
+    (property "Value" "GND" (at 17.78 60.325 0)
       (effects (font (size 1.27 1.27)))
     )
-    (property "Footprint" "" (at 20.955 55.245 0)
+    (property "Footprint" "" (at 17.78 55.245 0)
       (effects (font (size 1.27 1.27)) hide)
     )
-    (property "Datasheet" "" (at 20.955 55.245 0)
+    (property "Datasheet" "" (at 17.78 55.245 0)
       (effects (font (size 1.27 1.27)) hide)
     )
